File: Hardware/SparkFun_Qwiic_WAV_Trigger_Pro.kicad_sch (KiCad schematic)
At the start: 11 parts

Commit message: Changed board rev knockout to v02
Added VBUS voltage divider R26/R27 for VBUS detect input, STM32 PA9

Fixed reversed I2S SCK and SDA signals at STM32

JTAG debug connector pin 1 now connects to 3.3V

Added 2-pin header/jumper for pulling STM32 BOOT0 high

Changed trigger silkscreen labelling

Changed DEV/HST silkscreen label

Added date to all pages

Signed-off-by: Jamie Robertson <jrr@robertsonics.com>
Other:
- sheet CPU ports: added VBUS_DET; removed none
- sheet USB ports: added VBUS_DET; removed none
Changed lines of the file:
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@@
 	(title_block
 		(title "SparkFun Qwiic WAV Trigger Pro")
+		(date "2024-08-19")
 		(rev "1.0")
 		(company "Robertsonics / SparkFun")
@@
 		(pts
 			(xy 166.37 71.12) (xy 182.88 71.12)
+		)
+		(stroke
+			(width 0)
+			(type default)
+		)
+	)
+	(wire
+		(pts
+			(xy 97.79 74.93) (xy 114.3 74.93)
 		)
 		(stroke
@@
 			)
 		)
+		(pin "VBUS_DET" input
+			(at 114.3 74.93 180)
+			(effects
+				(font
+					(size 1.27 1.27)
+				)
+				(justify left)
+			)
+		)
 		(instances
 			(project "SparkFun_Qwiic_WAV_Trigger_Pro"
@@
 			(effects
 				(font
+					(size 1.27 1.27)
+				)
+				(justify right)
+			)
+		)
+		(pin "VBUS_DET" output
+			(at 97.79 74.93 0)
+			(effects
+				(font

Commit message: Add ordering instructions. Panelize.
Parts:
- added U8: ~, SparkFun-Aesthetic:Ordering_Instructions, symbol SparkFun-Aesthetic:Ordering_Instructions
Changed lines of the file:
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@@
 		)
 		(instances
-			(project "SparkFun_Qwiic_WAV_Trigger_Pro"
+			(project "SparkFun_Qwiic_WAV_Trigger_Pro_panelized"
 				(path "/4c0b78e3-6801-43aa-85ca-70880324c2bd"
 					(reference "G1")
@@
 		)
 		(instances
-			(project "SparkFun_Qwiic_WAV_Trigger_Pro"
+			(project "SparkFun_Qwiic_WAV_Trigger_Pro_panelized"
 				(path "/4c0b78e3-6801-43aa-85ca-70880324c2bd"
 					(reference "ST2")
@@
 		)
 		(instances
-			(project "SparkFun_Qwiic_WAV_Trigger_Pro"
+			(project "SparkFun_Qwiic_WAV_Trigger_Pro_panelized"
 				(path "/4c0b78e3-6801-43aa-85ca-70880324c2bd"
 					(reference "ST3")
@@
 		)
 		(instances
-			(project "SparkFun_Qwiic_WAV_Trigger_Pro"
+			(project "SparkFun_Qwiic_WAV_Trigger_Pro_panelized"
 				(path "/4c0b78e3-6801-43aa-85ca-70880324c2bd"
 					(reference "G3")
@@
 		)
 		(instances
-			(project "SparkFun_Qwiic_WAV_Trigger_Pro"
+			(project "SparkFun_Qwiic_WAV_Trigger_Pro_panelized"
 				(path "/4c0b78e3-6801-43aa-85ca-70880324c2bd"
 					(reference "FID2")
+					(unit 1)
+				)
+			)
+		)
+	)
+	(symbol
+		(lib_id "SparkFun-Aesthetic:Ordering_Instructions")
+		(at 223.52 175.26 0)
+		(unit 1)
+		(exclude_from_sim no)
+		(in_bom yes)
+		(on_board yes)
+		(dnp no)
+		(fields_autoplaced yes)
+		(property "Reference" "U8"
+			(at 223.52 172.72 0)
+			(effects
+				(font
+					(size 1.27 1.27)
+				)
+				(hide yes)
+			)
+		)
+		(property "Value" "~"
+			(at 223.52 175.26 0)
+			(effects
+				(font
+					(size 1.27 1.27)
+				)
+				(hide yes)
+			)
+		)
+		(property "Footprint" "SparkFun-Aesthetic:Ordering_Instructions"
+			(at 223.52 179.07 0)
+			(effects
+				(font
+					(size 1.27 1.27)
+				)
+				(hide yes)
+			)
+		)
+		(property "Datasheet" ""
+			(at 223.52 175.26 0)
+			(effects
+				(font
+					(size 1.27 1.27)
+				)
+				(hide yes)
+			)
+		)
+		(property "Description" ""
+			(at 223.52 175.26 0)
+			(effects
+				(font
+					(size 1.27 1.27)
+				)
+				(hide yes)
+			)
+		)
+		(instances
+			(project "SparkFun_Qwiic_WAV_Trigger_Pro_panelized"
+				(path "/4c0b78e3-6801-43aa-85ca-70880324c2bd"
+					(reference "U8")
 					(unit 1)
 				)
@@
 		)
 		(instances
-			(project "SparkFun_Qwiic_WAV_Trigger_Pro"
+			(project "SparkFun_Qwiic_WAV_Trigger_Pro_panelized"
 				(path "/4c0b78e3-6801-43aa-85ca-70880324c2bd"
 					(reference "ST1")
@@
 		)
 		(instances
-			(project "SparkFun_Qwiic_WAV_Trigger_Pro"
+			(project "SparkFun_Qwiic_WAV_Trigger_Pro_panelized"
 				(path "/4c0b78e3-6801-43aa-85ca-70880324c2bd"
 					(reference "G4")
@@
 		)
 		(instances
-			(project "SparkFun_Qwiic_WAV_Trigger_Pro"
+			(project "SparkFun_Qwiic_WAV_Trigger_Pro_panelized"
 				(path "/4c0b78e3-6801-43aa-85ca-70880324c2bd"
 					(reference "FID4")
@@
 		)
 		(instances
-			(project "SparkFun_Qwiic_WAV_Trigger_Pro"
+			(project "SparkFun_Qwiic_WAV_Trigger_Pro_panelized"
 				(path "/4c0b78e3-6801-43aa-85ca-70880324c2bd"
 					(reference "FID3")
@@
 		)
 		(instances
-			(project "SparkFun_Qwiic_WAV_Trigger_Pro"
+			(project "SparkFun_Qwiic_WAV_Trigger_Pro_panelized"
 				(path "/4c0b78e3-6801-43aa-85ca-70880324c2bd"
 					(reference "ST4")
@@
 		)
 		(instances
-			(project "SparkFun_Qwiic_WAV_Trigger_Pro"
+			(project "SparkFun_Qwiic_WAV_Trigger_Pro_panelized"
 				(path "/4c0b78e3-6801-43aa-85ca-70880324c2bd"
 					(reference "FID1")
@@
 		)
 		(instances
-			(project "SparkFun_Qwiic_WAV_Trigger_Pro"
+			(project "SparkFun_Qwiic_WAV_Trigger_Pro_panelized"
 				(path "/4c0b78e3-6801-43aa-85ca-70880324c2bd"
 					(page "3")
@@
 		)
 		(instances
-			(project "SparkFun_Qwiic_WAV_Trigger_Pro"
+			(project "SparkFun_Qwiic_WAV_Trigger_Pro_panelized"
 				(path "/4c0b78e3-6801-43aa-85ca-70880324c2bd"
 					(page "2")
@@
 		)
 		(instances
-			(project "SparkFun_Qwiic_WAV_Trigger_Pro"
+			(project "SparkFun_Qwiic_WAV_Trigger_Pro_panelized"
 				(path "/4c0b78e3-6801-43aa-85ca-70880324c2bd"
 					(page "4")
